Commit message: Added demo urdf, update cmake, launch, and package files

File: src/trike/urdf/trike.urdf (robot description, URDF)
Before this commit: robot trike, 6 links, 5 joints
Links:
- link front_frame: geometry visual box size=2.44 0.1 0.1
- link front_left_wheel: geometry visual cylinder length=0.076 radius=0.24
- link front_right_wheel: geometry visual cylinder length=0.076 radius=0.24
- link rear_wheel: geometry visual cylinder length=0.076 radius=0.24
Joints:
- joint frame_joint: origin xyz=${wheelbase} 0 0 -> xyz=1.22 0 0
- joint front_left_wheel_joint: origin xyz=${wheelbase} ${frame_width / 2} -${wheel_radius} -> xyz=1.22 0.305 -0.24
- joint front_right_wheel_joint: origin xyz=${wheelbase} -${frame_width / 2} -${wheel_radius} -> xyz=1.22 -0.305 -0.24
- joint rear_wheel_joint: origin xyz=0 0 -${wheel_radius} -> xyz=0 0 -0.24
- joint steering_joint: limit lower=-${steering_angle_max} upper=${steering_angle_max} effort=1.0 velocity=1.0 -> lower=-0.96 upper=0.96 effort=1.0 velocity=1.0; origin xyz=${wheelbase} 0 0.1 -> xyz=1.22 0 0.1
