Commit message: added urdf

File: src/trike/urdf/ackerman.xacro (robot description, xacro)
@@ -9,18 +9,19 @@
     </visual>
   </link>
-  <joint name="base_joint" type="fixed">
-    <parent link="base_link"/>
-    <child link="chassis"/>
-  </joint>
+ <joint name="base_joint" type="fixed">
+  <parent link="base_link"/>
+  <child link="chassis"/>
+  <origin xyz="0 0 0.735" rpy="0 0 0"/>
+ </joint>
   <link name="chassis">
     <collision>
       <origin xyz="0 0 0" rpy="0 0 0"/>
       <geometry>
-        <box size="2.4 0.58 1.06"/>
-      </geometry>
-    </collision>
-    <visual>
-      <origin xyz="0 0 -0.13" rpy="0 0 0"/> <geometry>
-        <box size="2.4 0.58 0.8"/>
+        <box size="2.4 0.58 0.86"/>
+      </geometry>
+    </collision>
+    <visual>
+      <origin xyz="0 0 0" rpy="0 0 0"/> <geometry>
+        <box size="2.4 0.58 0.86"/>
       </geometry>
       <material name="orange"/>
@@ -104,5 +105,5 @@
     <parent link="chassis"/>
     <child link="right_wheel_assembly"/>
-    <origin xyz="0.0 0.29 -0.21" rpy="0 0 0" /> <axis xyz="0 0 1" rpy="0 0 0" />
+    <origin xyz="0.45 0.29 -0.48" rpy="0 0 0" /> <axis xyz="0 0 1" rpy="0 0 0" />
     <limit effort="100" velocity="1" lower="-1" upper="1"/>
     <dynamics damping="0.0" friction="0.0"/>
@@ -197,5 +198,5 @@
     <parent link="chassis"/>
     <child link="left_wheel_assembly"/>
-    <origin xyz="0.45 -0.29 -0.21" rpy="0 0 0" /> <axis xyz="0 0 1" rpy="0 0 0" />
+    <origin xyz="0.45 -0.29 -0.48" rpy="0 0 0" /> <axis xyz="0 0 1" rpy="0 0 0" />
     <limit effort="100" velocity="1" lower="-1" upper="1"/>
     <dynamics damping="0.0" friction="0.0"/>
@@ -229,70 +230,46 @@
     </actuator>
   </transmission>
-  <link name="rear_right_wheel">
-    <collision>
-      <origin xyz="0 0 0" rpy="0 1.5708 1.5708" />
-      <geometry>
-        <cylinder length="0.05" radius="0.25"/>
-      </geometry>
-    </collision>
-    <visual>
-      <origin xyz="0 0 0" rpy="0 1.5708 1.5708" />
-      <geometry>
-        <cylinder length="0.05" radius="0.25"/>
-      </geometry>
-      <material name="black"/> </visual>
-    <inertial>
-      <origin xyz="0 0 0" rpy="0 1.5708 1.5708" />
-      <mass value="0.2"/>
-      <inertia ixx="0.001" ixy="0" ixz="0" iyy="0.001" iyz="0" izz="0.002"/>
-    </inertial>
-  </link>
-  <joint name="rear_right_wheel_joint" type="continuous">
-    <parent link="chassis"/>
-    <child link="rear_right_wheel"/>
-    <origin xyz="-0.9 0.29 -0.21" rpy="0 0 0" /> <axis xyz="0 1 0" rpy="0 0 0" />
-    <limit effort="100" velocity="50"/>
-    <dynamics damping="0.0" friction="0.0"/>
-  </joint>
-  <gazebo reference="rear_right_wheel">
-    <mu1 value="2.0"/>
-    <mu2 value="2.0"/>
-    <kp value="10000000.0" />
-    <kd value="1.0" />
-    <fdir1 value="0 1 0"/>
-    <material>Gazebo/Blue</material> </gazebo>
-  <link name="rear_left_wheel">
-    <collision>
-      <origin xyz="0 0 0" rpy="0 1.5708 1.5708" />
-      <geometry>
-        <cylinder length="0.05" radius="0.25"/>
-      </geometry>
-    </collision>
-    <visual>
-      <origin xyz="0 0 0" rpy="0 1.5708 1.5708" />
-      <geometry>
-        <cylinder length="0.05" radius="0.25"/>
-      </geometry>
-      <material name="black"/> </visual>
-    <inertial>
-      <origin xyz="0 0 0" rpy="0 1.5708 1.5708" />
-      <mass value="0.2"/>
-      <inertia ixx="0.001" ixy="0" ixz="0" iyy="0.001" iyz="0" izz="0.002"/>
-    </inertial>
-  </link>
-  <joint name="rear_left_wheel_joint" type="continuous">
-    <parent link="chassis"/>
-    <child link="rear_left_wheel"/>
-    <origin xyz="-0.9 -0.29 -0.21" rpy="0 0 0" /> <axis xyz="0 1 0" rpy="0 0 0" />
-    <limit effort="100" velocity="50"/>
-    <dynamics damping="0.0" friction="0.0"/>
-  </joint>
-  <gazebo reference="rear_left_wheel">
-    <mu1 value="2.0"/>
-    <mu2 value="2.0"/>
-    <kp value="10000000.0" />
-    <kd value="1.0" />
-    <fdir1 value="0 1 0"/>
-    <material>Gazebo/Blue</material> </gazebo>
+<link name="rear_wheel">
+      <collision>
+          <origin xyz="0 0 0" rpy="0 1.5708 1.5708" />
+          <geometry>
+              <cylinder length="0.05" radius="0.25"/>
+          </geometry>
+      </collision>
+      <visual>
+          <origin xyz="0 0 0" rpy="0 1.5708 1.5708" />
+          <geometry>
+                <cylinder length="0.05" radius="0.25"/>
+          </geometry>
+          <material name="black"/> </visual>
+      <inertial>
+          <origin xyz="0 0 0" rpy="0 1.5708 1.5708" />
+          <mass value="0.2"/>
+          <inertia ixx="0.001" ixy="0" ixz="0" iyy="0.001" iyz="0" izz="0.002"/>
+      </inertial>
+  </link>
+  <joint name="rear_wheel_joint" type="continuous">
+      <parent link="chassis"/>
+      <child link="rear_wheel"/>
+      <origin xyz="-0.9 0 -0.48" rpy="0 0 0" />
+      <axis xyz="0 1 0" rpy="0 0 0" />
+      <limit effort="100" velocity="50"/>
+      <dynamics damping="0.0" friction="0.0"/>
+  </joint>
+  <gazebo reference="rear_wheel">
+      <mu1 value="2.0"/>
+      <mu2 value="2.0"/>
+      <kp value="10000000.0" />
+      <kd value="1.0" />
+      <fdir1 value="0 1 0"/>
+      <material>Gazebo/Blue</material> </gazebo>
+  <transmission name="trans_rear_wheel_rotate">
+    <type>transmission_interface/SimpleTransmission</type>
+    <joint name="rear_wheel_joint">
+      <hardwareInterface>EffortJointInterface</hardwareInterface> </joint>
+    <actuator name="motor_rear_wheel_rotate">
+      <hardwareInterface>EffortJointInterface</hardwareInterface> <mechanicalReduction>1</mechanicalReduction>
+    </actuator>
+  </transmission>
   <gazebo>
     <plugin name="gazebo_ros_control" filename="libgazebo_ros_control.so">
